File: CurrentSinkOrSwim.sch (KiCad schematic (older format))
At the start: 10 parts

Commit message: Add spice simulation, and also a couple part numbers for resister and FET
Parts:
- Q?: value Q_NMOS_DGS -> BUK9575; MPN (none) -> BUK9575-100A,127
- R?: value R -> .1; MPN (none) -> AC01000001007JA100
Changed lines of the file:
@@
 P 6450 3600
 F 0 "Q?" H 6750 3650 50  0000 R CNN
-F 1 "Q_NMOS_DGS" H 7100 3550 50  0000 R CNN
+F 1 "BUK9575" H 7100 3550 50  0000 R CNN
 F 2 "" H 6650 3700 50  0000 C CNN
 F 3 "" H 6450 3600 50  0000 C CNN
+F 4 "BUK9575-100A,127" H 6450 3600 60  0001 C CNN "MPN"
 	1    6450 3600
 	1    0    0    -1
@@
 P 6550 4450
 F 0 "R?" V 6630 4450 50  0000 C CNN
-F 1 "R" V 6550 4450 50  0000 C CNN
+F 1 ".1" V 6550 4450 50  0000 C CNN
 F 2 "" V 6480 4450 50  0000 C CNN
 F 3 "" H 6550 4450 50  0000 C CNN
+F 4 "AC01000001007JA100" V 6550 4450 60  0001 C CNN "MPN"
 	1    6550 4450
 	1    0    0    -1

Commit message: Added variable regulator to circuit
Parts:
- removed U?: TC1016, symbol TC1016
- added C?: C, symbol C
- added P?: CONN_01X03, symbol CONN_01X03
- added P?: CONN_01X02, symbol CONN_01X02
- added R?: 0, symbol R
- added R?: 27k, symbol R
- added R?: 21.6k, symbol R
- added U?: LM2931D-R, symbol LM2931D-R
Connections:
- net labels added: 2.7V
- wire segments 22 -> 43
Other:
- note added: "Battery Pack"
- note added: "Current Sink Input"
- moved on the sheet: C?, P?, Q?
