File: CurrentControl.sch (KiCad schematic (older format))
At the start: 7 parts

Commit message: Annotation completed
Parts:
- gave numbers to parts that had none: 7
Changed lines of the file:
@@
 $EndDescr
 $Comp
-L LMV358 U?
+L LMV358 U201
 U 1 1 57DA1673
 P 5400 3400
-F 0 "U?" H 5350 3600 50  0000 L CNN
+F 0 "U201" H 5350 3600 50  0000 L CNN
 F 1 "LMV358" H 5350 3150 50  0000 L CNN
 F 2 "" H 5400 3400 50  0000 C CNN
@@
 $EndComp
 $Comp
-L Q_NMOS_DGS Q?
+L Q_NMOS_DGS Q201
 U 1 1 57DA1681
 P 6750 3400
-F 0 "Q?" H 7050 3450 50  0000 R CNN
+F 0 "Q201" H 7050 3450 50  0000 R CNN
 F 1 "BUK9575" H 7400 3350 50  0000 R CNN
 F 2 "" H 6950 3500 50  0000 C CNN
@@
 $EndComp
 $Comp
-L R R?
+L R R201
 U 1 1 57DA1688
 P 4300 4350
-F 0 "R?" V 4380 4350 50  0000 C CNN
+F 0 "R201" V 4380 4350 50  0000 C CNN
 F 1 "R" V 4300 4350 50  0000 C CNN
 F 2 "" V 4230 4350 50  0000 C CNN
@@
 $EndComp
 $Comp
-L R R?
+L R R203
 U 1 1 57DA1690
 P 6850 4250
-F 0 "R?" V 6930 4250 50  0000 C CNN
+F 0 "R203" V 6930 4250 50  0000 C CNN
 F 1 ".1" V 6850 4250 50  0000 C CNN
 F 2 "" V 6780 4250 50  0000 C CNN
@@
 $EndComp
 $Comp
-L GND #PWR?
+L GND #PWR202
 U 1 1 57DA1697
 P 5300 3700
-F 0 "#PWR?" H 5300 3450 50  0001 C CNN
+F 0 "#PWR202" H 5300 3450 50  0001 C CNN
 F 1 "GND" H 5300 3550 50  0000 C CNN
 F 2 "" H 5300 3700 50  0000 C CNN
@@
 $EndComp
 $Comp
-L POT RV?
+L POT RV201
 U 1 1 57DA169D
 P 4300 3750
-F 0 "RV?" H 4300 3670 50  0000 C CNN
+F 0 "RV201" H 4300 3670 50  0000 C CNN
 F 1 "POT" H 4300 3750 50  0000 C CNN
 F 2 "" H 4300 3750 50  0000 C CNN
@@
 $EndComp
 $Comp
-L C C?
+L C C201
 U 1 1 57DA16A4
 P 4900 2750
-F 0 "C?" H 4925 2850 50  0000 L CNN
+F 0 "C201" H 4925 2850 50  0000 L CNN
 F 1 "C" H 4925 2650 50  0000 L CNN
 F 2 "" H 4938 2600 50  0000 C CNN
@@
 $EndComp
 $Comp
-L GND #PWR?
+L GND #PWR201
 U 1 1 57DA16AB
 P 4900 2900
-F 0 "#PWR?" H 4900 2650 50  0001 C CNN
+F 0 "#PWR201" H 4900 2650 50  0001 C CNN
 F 1 "GND" H 4900 2750 50  0000 C CNN
 F 2 "" H 4900 2900 50  0000 C CNN
@@
 Connection ~ 4900 2500
 $Comp
-L R R?
+L R R202
 U 1 1 57DA1A1C
 P 6050 3400
-F 0 "R?" V 6130 3400 50  0000 C CNN
+F 0 "R202" V 6130 3400 50  0000 C CNN
 F 1 "1k" V 6050 3400 50  0000 C CNN
 F 2 "" V 5980 3400 50  0000 C CNN

Commit message: Add initial layout
Parts:
- C201: footprint (none) -> Capacitors_SMD:C_0805
- Q201: footprint (none) -> TO_SOT_Packages_THT:TO-220_Neutral123_Vertical
- R201, R202: footprint (none) -> Resistors_SMD:R_0805
- R203: footprint (none) -> Resistors_ThroughHole:Resistor_Horizontal_RM15mm
- RV201: footprint (none) -> Potentiometers:Potentiometer_WirePads_largePads
- U201: value LMV358 -> LMV358IDT; footprint (none) -> SMD_Packages:SOIC-8-N
Changed lines of the file:
@@
 P 5400 3400
 F 0 "U201" H 5350 3600 50  0000 L CNN
-F 1 "LMV358" H 5350 3150 50  0000 L CNN
-F 2 "" H 5400 3400 50  0000 C CNN
-F 3 "" H 5400 3400 50  0000 C CNN
+F 1 "LMV358IDT" H 5350 3150 50  0000 L CNN
+F 2 "SMD_Packages:SOIC-8-N" H 5400 3400 50  0001 C CNN
+F 3 "http://www.st.com/content/ccc/resource/technical/document/datasheet/b9/d8/3b/8f/a1/8f/46/01/CD00079372.pdf/files/CD00079372.pdf/jcr:content/translations/en.CD00079372.pdf" H 5400 3400 50  0001 C CNN
 	1    5400 3400
 	1    0    0    -1
@@
 F 0 "Q201" H 7050 3450 50  0000 R CNN
 F 1 "BUK9575" H 7400 3350 50  0000 R CNN
-F 2 "" H 6950 3500 50  0000 C CNN
+F 2 "TO_SOT_Packages_THT:TO-220_Neutral123_Vertical" H 6950 3500 50  0001 C CNN
 F 3 "http://www.nxp.com/documents/data_sheet/BUK9575-100A.pdf" H 6750 3400 50  0001 C CNN
 F 4 "BUK9575-100A,127" H 6750 3400 60  0001 C CNN "MPN"
@@
 F 0 "R201" V 4380 4350 50  0000 C CNN
 F 1 "R" V 4300 4350 50  0000 C CNN
-F 2 "" V 4230 4350 50  0000 C CNN
+F 2 "Resistors_SMD:R_0805" V 4230 4350 50  0001 C CNN
 F 3 "" H 4300 4350 50  0000 C CNN
 	1    4300 4350
@@
 F 0 "R203" V 6930 4250 50  0000 C CNN
 F 1 ".1" V 6850 4250 50  0000 C CNN
-F 2 "" V 6780 4250 50  0000 C CNN
+F 2 "Resistors_ThroughHole:Resistor_Horizontal_RM15mm" V 6780 4250 50  0001 C CNN
 F 3 "http://www.mouser.com/ds/2/427/acseries-222859.pdf" H 6850 4250 50  0001 C CNN
 F 4 "AC01000001007JA100" V 6850 4250 60  0001 C CNN "MPN"
@@
 $EndComp
 $Comp
-L GND #PWR202
+L GND #PWR03
 U 1 1 57DA1697
 P 5300 3700
-F 0 "#PWR202" H 5300 3450 50  0001 C CNN
+F 0 "#PWR03" H 5300 3450 50  0001 C CNN
 F 1 "GND" H 5300 3550 50  0000 C CNN
 F 2 "" H 5300 3700 50  0000 C CNN
@@
 F 0 "RV201" H 4300 3670 50  0000 C CNN
 F 1 "POT" H 4300 3750 50  0000 C CNN
-F 2 "" H 4300 3750 50  0000 C CNN
+F 2 "Potentiometers:Potentiometer_WirePads_largePads" H 4300 3750 50  0001 C CNN
 F 3 "" H 4300 3750 50  0000 C CNN
 	1    4300 3750
@@
 F 0 "C201" H 4925 2850 50  0000 L CNN
 F 1 "C" H 4925 2650 50  0000 L CNN
-F 2 "" H 4938 2600 50  0000 C CNN
+F 2 "Capacitors_SMD:C_0805" H 4938 2600 50  0001 C CNN
 F 3 "" H 4900 2750 50  0000 C CNN
 	1    4900 2750
@@
 $EndComp
 $Comp
-L GND #PWR201
+L GND #PWR04
 U 1 1 57DA16AB
 P 4900 2900
-F 0 "#PWR201" H 4900 2650 50  0001 C CNN
+F 0 "#PWR04" H 4900 2650 50  0001 C CNN
 F 1 "GND" H 4900 2750 50  0000 C CNN
 F 2 "" H 4900 2900 50  0000 C CNN
@@
 F 0 "R202" V 6130 3400 50  0000 C CNN
 F 1 "1k" V 6050 3400 50  0000 C CNN
-F 2 "" V 5980 3400 50  0000 C CNN
+F 2 "Resistors_SMD:R_0805" V 5980 3400 50  0001 C CNN
 F 3 "" H 6050 3400 50  0000 C CNN
 	1    6050 3400

Commit message: Add heat sink footprint
Parts:
- added P201: CONN_01X01, current:FA-T220-38E-ND, symbol CONN_01X01
Changed lines of the file:
@@
 	4450 1550 4450 3750
-Wire Wire Line
-	6850 1750 6850 3200
 Wire Wire Line
 	5300 2500 5300 3100
@@
 Text HLabel 7400 4800 2    60   Input ~ 0
 Current_Sink-
+$Comp
+L CONN_01X01 P201
+U 1 1 57E5EC8F
+P 7750 2900
+F 0 "P201" H 7750 3000 50  0000 C CNN
+F 1 "CONN_01X01" V 7850 2900 50  0000 C CNN
+F 2 "current:FA-T220-38E-ND" H 7750 2900 50  0001 C CNN
+F 3 "http://www.ohmite.com/cat/sink_f_r.pdf" H 7750 2900 50  0001 C CNN
+F 4 "FA-T220-38E-ND" H 7750 2900 60  0001 C CNN "MPN"
+	1    7750 2900
+	1    0    0    -1
+$EndComp
+Wire Wire Line
+	6850 1750 6850 3200
 $EndSCHEMATC

Commit message: Remove extra erroneus LMV358
Parts:
- U201: value LMV358IDT -> LMV358; MPN (none) -> LMV358IDT
Changed lines of the file:
@@
 P 5400 3400
 F 0 "U201" H 5350 3600 50  0000 L CNN
-F 1 "LMV358IDT" H 5350 3150 50  0000 L CNN
+F 1 "LMV358" H 5350 3150 50  0000 L CNN
 F 2 "SMD_Packages:SOIC-8-N" H 5400 3400 50  0001 C CNN
 F 3 "http://www.st.com/content/ccc/resource/technical/document/datasheet/b9/d8/3b/8f/a1/8f/46/01/CD00079372.pdf/files/CD00079372.pdf/jcr:content/translations/en.CD00079372.pdf" H 5400 3400 50  0001 C CNN
+F 4 "LMV358IDT" H 5400 3400 60  0001 C CNN "MPN"
 	1    5400 3400
 	1    0    0    -1

Commit message: Add potentiometers
Parts:
- RV201: footprint Potentiometers:Potentiometer_WirePads_largePads -> current:P090L-02F25BR10K; MPN (none) -> P090L-02F25BR10K
Changed lines of the file:
@@
 F 0 "RV201" H 4300 3670 50  0000 C CNN
 F 1 "POT" H 4300 3750 50  0000 C CNN
-F 2 "Potentiometers:Potentiometer_WirePads_largePads" H 4300 3750 50  0001 C CNN
-F 3 "" H 4300 3750 50  0000 C CNN
+F 2 "current:P090L-02F25BR10K" H 4300 3750 50  0001 C CNN
+F 3 "http://www.bitechnologies.com/pdfs/p090.pdf" H 4300 3750 50  0001 C CNN
+F 4 "P090L-02F25BR10K" H 4300 3750 60  0001 C CNN "MPN"
 	1    4300 3750
 	0    1    1    0

Commit message: Fixed divider resistors and found values
Parts:
- R201: value R -> 68k
- RV201: value POT -> 10k
Connections:
- net 2.7V: now also R201.1; no longer RV201.2
- net Current_Sink-: now also RV201.2; no longer R201.2
- net at RV201.1: now also R201.2, U201.3 (+)
- now unconnected: RV201.3
Other:
- moved on the sheet: R201, RV201
Changed lines of the file:
@@
 L R R201
 U 1 1 57DA1688
-P 4300 4350
-F 0 "R201" V 4380 4350 50  0000 C CNN
-F 1 "R" V 4300 4350 50  0000 C CNN
-F 2 "Resistors_SMD:R_0805" V 4230 4350 50  0001 C CNN
-F 3 "" H 4300 4350 50  0000 C CNN
-	1    4300 4350
+P 4450 3900
+F 0 "R201" V 4530 3900 50  0000 C CNN
+F 1 "68k" V 4450 3900 50  0000 C CNN
+F 2 "Resistors_SMD:R_0805" V 4380 3900 50  0001 C CNN
+F 3 "" H 4450 3900 50  0000 C CNN
+	1    4450 3900
 	1    0    0    -1
 $EndComp
@@
 L POT RV201
 U 1 1 57DA169D
-P 4300 3750
-F 0 "RV201" H 4300 3670 50  0000 C CNN
-F 1 "POT" H 4300 3750 50  0000 C CNN
-F 2 "current:P090L-02F25BR10K" H 4300 3750 50  0001 C CNN
-F 3 "http://www.bitechnologies.com/pdfs/p090.pdf" H 4300 3750 50  0001 C CNN
-F 4 "P090L-02F25BR10K" H 4300 3750 60  0001 C CNN "MPN"
-	1    4300 3750
+P 4450 4500
+F 0 "RV201" H 4450 4420 50  0000 C CNN
+F 1 "10k" H 4450 4500 50  0000 C CNN
+F 2 "current:P090L-02F25BR10K" H 4450 4500 50  0001 C CNN
+F 3 "http://www.bitechnologies.com/pdfs/p090.pdf" H 4450 4500 50  0001 C CNN
+F 4 "P090L-02F25BR10K" H 4450 4500 60  0001 C CNN "MPN"
+	1    4450 4500
 	0    1    1    0
 $EndComp
@@
 Connection ~ 6850 4000
 Wire Wire Line
-	4300 3900 4300 4200
-Wire Wire Line
 	5100 3300 4700 3300
 Wire Wire Line
-	4700 3300 4700 4100
+	4700 3300 4700 4200
 Wire Wire Line
-	4700 4100 4300 4100
-Connection ~ 4300 4100
-Wire Wire Line
-	4300 4500 6850 4500
+	4600 4500 6850 4500
 Connection ~ 6850 4500
 Wire Wire Line
@@
 Wire Wire Line
 	6850 1750 6850 3200
+Wire Wire Line
+	4450 4350 4450 4050
+Wire Wire Line
+	4700 4200 4450 4200
+Connection ~ 4450 4200
 $EndSCHEMATC

Commit message: Lets try layout one more time. Starting layout from scratch
Parts:
- Q201: symbol Q_NMOS_DGS -> Q_NMOS_GDS
Connections:
- net Current_Sink+: now also Q201.2 (D); no longer Q201.1 (D)
- net FetGate: now also Q201.1 (G); no longer Q201.2 (G)
Changed lines of the file:
@@
 $EndComp
 $Comp
-L Q_NMOS_DGS Q201
+L Q_NMOS_GDS Q201
 U 1 1 57DA1681
 P 6750 3400

Commit message: Version 3 of the layout
Parts:
- removed C201: C, Capacitors_SMD:C_0805, symbol C
Connections:
- net at R202.2: now also U201.7; no longer U201.1
- net at Q201.3 (S), R203.1: now also U201.6 (-); no longer U201.2 (-)
- net at R201.2, RV201.1: now also U201.5 (+); no longer U201.3 (+)
Changed lines of the file:
@@
 $Comp
 L LMV358 U201
-U 1 1 57DA1673
+U 2 1 57DA1673
 P 5400 3400
 F 0 "U201" H 5350 3600 50  0000 L CNN
@@
 F 3 "http://www.st.com/content/ccc/resource/technical/document/datasheet/b9/d8/3b/8f/a1/8f/46/01/CD00079372.pdf/files/CD00079372.pdf/jcr:content/translations/en.CD00079372.pdf" H 5400 3400 50  0001 C CNN
 F 4 "LMV358IDT" H 5400 3400 60  0001 C CNN "MPN"
-	1    5400 3400
+	2    5400 3400
 	1    0    0    -1
 $EndComp
@@
 $EndComp
 $Comp
-L C C201
-U 1 1 57DA16A4
-P 4900 2750
-F 0 "C201" H 4925 2850 50  0000 L CNN
-F 1 "C" H 4925 2650 50  0000 L CNN
-F 2 "Capacitors_SMD:C_0805" H 4938 2600 50  0001 C CNN
-F 3 "" H 4900 2750 50  0000 C CNN
-	1    4900 2750
-	1    0    0    -1
+L R R202
+U 1 1 57DA1A1C
+P 6050 3400
+F 0 "R202" V 6130 3400 50  0000 C CNN
+F 1 "1k" V 6050 3400 50  0000 C CNN
+F 2 "Resistors_SMD:R_0805" V 5980 3400 50  0001 C CNN
+F 3 "" H 6050 3400 50  0000 C CNN
+	1    6050 3400
+	0    1    1    0
 $EndComp
+Text GLabel 3550 1550 0    60   Input ~ 0
+2.7V
+Text HLabel 7350 1750 2    60   Input ~ 0
+Current_Sink+
+Text HLabel 7350 1500 2    60   Input ~ 0
+FetGate
+Text HLabel 7400 4800 2    60   Input ~ 0
+Current_Sink-
 $Comp
-L GND #PWR04
-U 1 1 57DA16AB
-P 4900 2900
-F 0 "#PWR04" H 4900 2650 50  0001 C CNN
-F 1 "GND" H 4900 2750 50  0000 C CNN
-F 2 "" H 4900 2900 50  0000 C CNN
-F 3 "" H 4900 2900 50  0000 C CNN
-	1    4900 2900
+L CONN_01X01 P201
+U 1 1 57E5EC8F
+P 7750 2900
+F 0 "P201" H 7750 3000 50  0000 C CNN
+F 1 "CONN_01X01" V 7850 2900 50  0000 C CNN
+F 2 "current:FA-T220-38E-ND" H 7750 2900 50  0001 C CNN
+F 3 "http://www.ohmite.com/cat/sink_f_r.pdf" H 7750 2900 50  0001 C CNN
+F 4 "FA-T220-38E-ND" H 7750 2900 60  0001 C CNN "MPN"
+	1    7750 2900
 	1    0    0    -1
 $EndComp
@@
 Wire Wire Line
 	5300 2500 5300 3100
-Wire Wire Line
-	4450 2500 5300 2500
 Connection ~ 4450 2500
-Wire Wire Line
-	4900 2600 4900 2500
-Connection ~ 4900 2500
-$Comp
-L R R202
-U 1 1 57DA1A1C
-P 6050 3400
-F 0 "R202" V 6130 3400 50  0000 C CNN
-F 1 "1k" V 6050 3400 50  0000 C CNN
-F 2 "Resistors_SMD:R_0805" V 5980 3400 50  0001 C CNN
-F 3 "" H 6050 3400 50  0000 C CNN
-	1    6050 3400
-	0    1    1    0
-$EndComp
 Wire Wire Line
 	5700 3400 5900 3400
 Wire Wire Line
 	6200 3400 6550 3400
-Text GLabel 3550 1550 0    60   Input ~ 0
-2.7V
 Wire Wire Line
 	3550 1550 4450 1550
 Wire Wire Line
 	6850 1750 7350 1750
-Text HLabel 7350 1750 2    60   Input ~ 0
-Current_Sink+
 Wire Wire Line
 	6400 3400 6400 1500
@@
 	6400 1500 7350 1500
 Connection ~ 6400 3400
-Text HLabel 7350 1500 2    60   Input ~ 0
-FetGate
 Wire Wire Line
 	6850 4800 7400 4800
-Text HLabel 7400 4800 2    60   Input ~ 0
-Current_Sink-
-$Comp
-L CONN_01X01 P201
-U 1 1 57E5EC8F
-P 7750 2900
-F 0 "P201" H 7750 3000 50  0000 C CNN
-F 1 "CONN_01X01" V 7850 2900 50  0000 C CNN
-F 2 "current:FA-T220-38E-ND" H 7750 2900 50  0001 C CNN
-F 3 "http://www.ohmite.com/cat/sink_f_r.pdf" H 7750 2900 50  0001 C CNN
-F 4 "FA-T220-38E-ND" H 7750 2900 60  0001 C CNN "MPN"
-	1    7750 2900
-	1    0    0    -1
-$EndComp
 Wire Wire Line
 	6850 1750 6850 3200
 Wire Wire Line
-	4450 4350 4450 4050
+	4450 4050 4450 4350
 Wire Wire Line
 	4700 4200 4450 4200
 Connection ~ 4450 4200
+Wire Wire Line
+	4450 2500 5300 2500
 $EndSCHEMATC
