File: CurrentControl.sch (KiCad schematic (older format))
At the start: 7 parts, among them P201 CONN_01X01, Q201 BUK9575, U201 LMV358

Commit message: Add preliminary BOM
Parts:
- P201: value CONN_01X01 -> HeatSink
Changed lines of the file:
@@
 P 7750 2900
 F 0 "P201" H 7750 3000 50  0000 C CNN
-F 1 "CONN_01X01" V 7850 2900 50  0000 C CNN
+F 1 "HeatSink" V 7850 2900 50  0000 C CNN
 F 2 "current:FA-T220-38E-ND" H 7750 2900 50  0001 C CNN
 F 3 "http://www.ohmite.com/cat/sink_f_r.pdf" H 7750 2900 50  0001 C CNN

Commit message: Final schematic and BOM and layout
Parts:
- R201: MPN (none) -> RC0805JR-0768KL
- R202: MPN (none) -> RC0805JR-071KL
Changed lines of the file:
@@
 F 1 "68k" V 4450 3900 50  0000 C CNN
 F 2 "Resistors_SMD:R_0805" V 4380 3900 50  0001 C CNN
-F 3 "" H 4450 3900 50  0000 C CNN
+F 3 "http://www.yageo.com/NewPortal/yageodocoutput?fileName=/pdf/R-Chip/PYu-RC_Group_51_RoHS_L_4.pdf" H 4450 3900 50  0001 C CNN
+F 4 "RC0805JR-0768KL" V 4450 3900 60  0001 C CNN "MPN"
 	1    4450 3900
 	1    0    0    -1
@@
 F 1 "1k" V 6050 3400 50  0000 C CNN
 F 2 "Resistors_SMD:R_0805" V 5980 3400 50  0001 C CNN
-F 3 "" H 6050 3400 50  0000 C CNN
+F 3 "http://www.yageo.com/NewPortal/yageodocoutput?fileName=/pdf/R-Chip/PYu-RC_Group_51_RoHS_L_4.pdf" H 6050 3400 50  0001 C CNN
+F 4 "RC0805JR-071KL" V 6050 3400 60  0001 C CNN "MPN"
 	1    6050 3400
 	0    1    1    0
