File: CurrentSinkOrSwim.kicad_pcb (KiCad board)
At the start: 2 copper layers, 41.7 x 51.6 mm, 22 parts, among them P101 CONN_01X02, P102 CONN_01X03, P103 CONN_01X02, P201 CONN_01X01, Q201 BUK9575, U201 LMV358, U401 LM2931

Commit message: Add gerber files
Parts:
- moved C401 4.47 mm to (163.9, 70.7), turned to 90 degrees
- moved C402 4.43 mm to (157.5, 70.7), turned to 90 degrees
Other:
- board text added: "Vin"
- board text added: "gnd"
Changed lines of the file:
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@@
     (area 123.76178 39.968099 206.830372 96.234308)
     (thickness 1.6)
-    (drawings 4)
+    (drawings 19)
     (tracks 125)
     (zones 0)
@@
   )
   (module Capacitors_SMD:C_0805 (layer B.Cu)
-    (at 167.12184 73.74636)
+    (at 163.90112 70.65264 90)
     (descr "Capacitor SMD 0805, reflow soldering, AVX (see smccp.pdf)")
     (tags "capacitor 0805")
     (attr smd)
-    (fp_text reference C401 (at 0.10668 -1.94056) (layer B.SilkS)
+    (fp_text reference C401 (at 0.10668 -1.94056 90) (layer B.SilkS)
       (effects (font (size 1 1) (thickness 0.15)) (justify mirror))
     )
-    (fp_text value C (at 0 -2.1) (layer B.Fab) hide
+    (fp_text value C (at 0 -2.1 90) (layer B.Fab) hide
       (effects (font (size 1 1) (thickness 0.15)) (justify mirror))
     )
@@
     (fp_line (start 0.5 0.85) (end -0.5 0.85) (layer B.SilkS) (width 0.15))
     (fp_line (start -0.5 -0.85) (end 0.5 -0.85) (layer B.SilkS) (width 0.15))
-    (pad 1 smd rect (at -1 0) (size 1 1.25) (layers B.Cu B.Paste B.Mask)
+    (pad 1 smd rect (at -1 0 90) (size 1 1.25) (layers B.Cu B.Paste B.Mask)
       (net 3 "/Power Regulation/Vin"))
-    (pad 2 smd rect (at 1 0) (size 1 1.25) (layers B.Cu B.Paste B.Mask)
+    (pad 2 smd rect (at 1 0 90) (size 1 1.25) (layers B.Cu B.Paste B.Mask)
       (net 2 GND))
     (model Capacitors_SMD.3dshapes/C_0805.wrl
@@
   )
   (module Capacitors_SMD:C_0805 (layer B.Cu)
-    (at 160.67024 73.74128)
+    (at 157.50032 70.65264 90)
     (descr "Capacitor SMD 0805, reflow soldering, AVX (see smccp.pdf)")
     (tags "capacitor 0805")
     (attr smd)
-    (fp_text reference C402 (at -0.04064 -1.80848) (layer B.SilkS)
+    (fp_text reference C402 (at -0.04064 -1.80848 90) (layer B.SilkS)
       (effects (font (size 1 1) (thickness 0.15)) (justify mirror))
     )
-    (fp_text value C (at 0 -2.1) (layer B.Fab) hide
+    (fp_text value C (at 0 -2.1 90) (layer B.Fab) hide
       (effects (font (size 1 1) (thickness 0.15)) (justify mirror))
     )
@@
     (fp_line (start 0.5 0.85) (end -0.5 0.85) (layer B.SilkS) (width 0.15))
     (fp_line (start -0.5 -0.85) (end 0.5 -0.85) (layer B.SilkS) (width 0.15))
-    (pad 1 smd rect (at -1 0) (size 1 1.25) (layers B.Cu B.Paste B.Mask)
+    (pad 1 smd rect (at -1 0 90) (size 1 1.25) (layers B.Cu B.Paste B.Mask)
       (net 1 2.7V))
-    (pad 2 smd rect (at 1 0) (size 1 1.25) (layers B.Cu B.Paste B.Mask)
+    (pad 2 smd rect (at 1 0 90) (size 1 1.25) (layers B.Cu B.Paste B.Mask)
       (net 2 GND))
     (model Capacitors_SMD.3dshapes/C_0805.wrl
@@
     (descr "Through hole pin header")
     (tags "pin header")
-    (fp_text reference P102 (at -3.81 3.81 360) (layer F.SilkS)
+    (fp_text reference P102 (at -0.08382 -2.66446 360) (layer F.SilkS)
       (effects (font (size 1 1) (thickness 0.15)))
     )
@@
     (tags "resistor 0805")
     (attr smd)
-    (fp_text reference R202 (at 3.71348 0.15748 360) (layer F.SilkS)
+    (fp_text reference R202 (at 3.45694 -0.30988 360) (layer F.SilkS)
       (effects (font (size 1 1) (thickness 0.15)))
     )
@@
     )
   )
+  (gr_line (start 175.85182 77.55128) (end 175.85182 77.6224) (angle 90) (layer F.SilkS) (width 0.2))
+  (gr_line (start 176.63922 76.76388) (end 175.85182 77.55128) (angle 90) (layer F.SilkS) (width 0.2))
+  (gr_line (start 177.37074 77.51826) (end 177.37074 77.56398) (angle 90) (layer F.SilkS) (width 0.2))
+  (gr_line (start 176.63922 76.78674) (end 177.37074 77.51826) (angle 90) (layer F.SilkS) (width 0.2))
+  (gr_line (start 176.63668 76.77912) (end 176.63922 76.77658) (angle 90) (layer F.SilkS) (width 0.2))
+  (gr_line (start 176.63668 78.7908) (end 176.63668 76.77912) (angle 90) (layer F.SilkS) (width 0.2))
+  (gr_text gnd (at 169.8117 73.7235) (layer F.SilkS)
+    (effects (font (size 1.5 1.5) (thickness 0.3)))
+  )
+  (gr_line (start 172.75302 81.10982) (end 172.8089 81.10982) (angle 90) (layer F.SilkS) (width 0.2))
+  (gr_line (start 171.85894 80.21574) (end 172.75302 81.10982) (angle 90) (layer F.SilkS) (width 0.2))
+  (gr_line (start 172.78096 79.26578) (end 172.86478 79.26578) (angle 90) (layer F.SilkS) (width 0.2))
+  (gr_line (start 171.831 80.21574) (end 172.78096 79.26578) (angle 90) (layer F.SilkS) (width 0.2))
+  (gr_line (start 172.55744 80.21574) (end 171.80306 80.21574) (angle 90) (layer F.SilkS) (width 0.2))
+  (gr_line (start 173.228 79.54518) (end 172.55744 80.21574) (angle 90) (layer F.SilkS) (width 0.2))
+  (gr_line (start 174.12208 79.54518) (end 173.228 79.54518) (angle 90) (layer F.SilkS) (width 0.2))
+  (gr_text Vin (at 175.85436 79.54518) (layer F.SilkS)
+    (effects (font (size 1.5 1.5) (thickness 0.3)))
+  )
   (gr_line (start 180.34 40.3098) (end 138.7094 40.3098) (angle 90) (layer Edge.Cuts) (width 0.1))
   (gr_line (start 180.34 91.948) (end 180.34 40.3098) (angle 90) (layer Edge.Cuts) (width 0.1))
   (gr_line (start 138.7348 91.948) (end 180.3654 91.948) (angle 90) (layer Edge.Cuts) (width 0.1))
   (gr_line (start 138.7094 40.3098) (end 138.7094 91.948) (angle 90) (layer Edge.Cuts) (width 0.1))
+  (segment (start 157.4673 73.7235) (end 157.4673 71.68566) (width 0.6096) (layer B.Cu) (net 1))
+  (segment (start 157.4673 71.68566) (end 157.50032 71.65264) (width 0.6096) (layer B.Cu) (net 1))
   (segment (start 141.33576 80.80248) (end 144.02384 80.80248) (width 0.6096) (layer B.Cu) (net 1))
   (segment (start 144.02384 80.80248) (end 151.26208 73.56424) (width 0.6096) (layer B.Cu) (net 1))
@@
   (segment (start 152.3619 73.7235) (end 151.26208 72.62368) (width 0.6096) (layer B.Cu) (net 1))
   (segment (start 157.48 75.565) (end 157.48 73.7362) (width 0.6096) (layer F.Cu) (net 1))
-  (segment (start 157.48508 73.74128) (end 159.67024 73.74128) (width 0.6096) (layer B.Cu) (net 1))
-  (segment (start 157.4673 73.7235) (end 157.48508 73.74128) (width 0.6096) (layer B.Cu) (net 1))
   (via (at 157.4673 73.7235) (size 1.143) (drill 0.762) (layers F.Cu B.Cu) (net 1))
   (segment (start 157.48 73.7362) (end 157.4673 73.7235) (width 0.6096) (layer F.Cu) (net 1))
@@
   (segment (start 160.0581 78.105) (end 157.48 78.105) (width 0.6096) (layer F.Cu) (net 2))
   (segment (start 161.3535 78.105) (end 160.7058 77.4573) (width 0.6096) (layer F.Cu) (net 2))
-  (segment (start 163.83 75.565) (end 163.83 74.0664) (width 0.6096) (layer F.Cu) (net 3))
-  (segment (start 164.19576 73.74636) (end 166.12184 73.74636) (width 0.6096) (layer B.Cu) (net 3))
-  (segment (start 164.1729 73.7235) (end 164.19576 73.74636) (width 0.6096) (layer B.Cu) (net 3))
-  (via (at 164.1729 73.7235) (size 1.143) (drill 0.762) (layers F.Cu B.Cu) (net 3))
-  (segment (start 163.83 74.0664) (end 164.1729 73.7235) (width 0.6096) (layer F.Cu) (net 3))
+  (segment (start 163.83 75.565) (end 163.83 73.79208) (width 0.6096) (layer F.Cu) (net 3))
+  (segment (start 163.90112 73.70064) (end 163.90112 71.65264) (width 0.6096) (layer B.Cu) (net 3))
+  (segment (start 163.81984 73.78192) (end 163.90112 73.70064) (width 0.6096) (layer B.Cu) (net 3))
+  (via (at 163.81984 73.78192) (size 1.143) (drill 0.762) (layers F.Cu B.Cu) (net 3))
+  (segment (start 163.83 73.79208) (end 163.81984 73.78192) (width 0.6096) (layer F.Cu) (net 3))
   (segment (start 170.434 80.264) (end 168.9608 80.264) (width 0.6096) (layer F.Cu) (net 3))
   (segment (start 167.1574 75.565) (end 163.83 75.565) (width 0.6096) (layer F.Cu) (net 3))
